Commit message: add semi final files

File: urdf/robot.xacro (robot description, xacro)
@@ -1,208 +1,186 @@
-<?xml version='1.0'?>
+<?xml version="1.0"?>
 <robot name="robot" xmlns:xacro="http://www.ros.org/wiki/xacro">
-<link name='chassis'>
-<pose>0 0 0.1 0 0 0</pose>
-<inertial>
-<mass value="5.0" />
-<origin xyz="0.0 0 0.1" rpy=" 0 0 0" />
-<inertia
-ixx="0.1" ixy="0" ixz="0"
-iyy="0.1" iyz="0"
-izz="0.1"
-/>
-</inertial>
-<collision name='collision'>
-<geometry>
-<box size=".4 .2 .1" />
-</geometry>
-</collision>
-<visual name='chassis_visual'>
-<origin xyz="0 0 0" rpy=" 0 0 0" />
-<geometry>
-<box size=".4 .2 .1" />
-</geometry>
-<material name="blue">
-<color rgba="0.0 0.0 1 1.0" />
-</material>
-</visual>
-<collision name='caster_collision'>
-<origin xyz="-0.15 0 -0.05" rpy=" 0 0 0" />
-<geometry>
-<sphere radius="0.05" />
-</geometry>
-</collision>
-<visual name='caster_visual'>
-<origin xyz="-0.15 0 -0.05" rpy=" 0 0 0" />
-<geometry>
-<sphere radius="0.05" />
-</geometry>
-</visual>
-<collision name='caster_front_collision'>
-<origin xyz="0.15 0 -0.05" rpy=" 0 0 0" />
-<geometry>
-<sphere radius="0.05" />
-</geometry>
-</collision>
-<visual name='caster_front_visual'>
-<origin xyz="0.15 0 -0.05" rpy=" 0 0 0" />
-<geometry>
-<sphere radius="0.05" />
-</geometry>
-</visual>
-</link>
-<link name="left_wheel">
-<collision name="collision">
-<origin xyz="0 0 0" rpy="0 1.5707 1.5707" />
-<geometry>
-<cylinder radius="0.1" length="0.05" />
-</geometry>
-</collision>
-<visual name="left_wheel_visual">
-<origin xyz="0 0 0" rpy="0 1.5707 1.5707" />
-<geometry>
-<cylinder radius="0.1" length="0.05" />
-</geometry>
-<material name="red">
-<color rgba="1 0.0 0.0 1.0" />
-</material>
-</visual>
-<inertial>
-<origin xyz="0 0 0" rpy="0 1.5707 1.5707" />
-<mass value="5" />
-<inertia
-ixx=".1" ixy="0.0" ixz="0.0"
-iyy=".1" iyz="0.0"
-izz=".1" />
-</inertial>
-</link>
-<link name="right_wheel">
-<collision name="collision">
-<origin xyz="0 0 0" rpy="0 1.5707 1.5707" />
-<geometry>
-<cylinder radius="0.1" length="0.05" />
-</geometry>
-</collision>
-<visual name="right_wheel_visual">
-<origin xyz="0 0 0" rpy="0 1.5707 1.5707" />
-<geometry>
-<cylinder radius="0.1" length="0.05" />
-</geometry>
-<material name="green">
-<color rgba="0.0 1 0.0 1.0" />
-</material>
-</visual>
-<inertial>
-<origin xyz="0 0 0" rpy="0 1.5707 1.5707" />
-<mass value="5" />
-<inertia
-ixx=".1" ixy="0.0" ixz="0.0"
-iyy=".1" iyz="0.0"
-izz=".1" />
-</inertial>
-</link>
-<joint type="continuous" name="left_wheel_hinge">
-<origin xyz="0 0.15 0" rpy="0 0 0" />
-<child link="left_wheel" />
-<parent link="chassis" />
-<axis xyz="0 1 0" rpy="0 0 0" />
-<joint_properties damping="0.0" friction="0.0" />
-</joint>
-<joint type="continuous" name="right_wheel_hinge">
-<origin xyz="0 -0.15 0" rpy="0 0 0" />
-<child link="right_wheel" />
-<parent link="chassis" />
-<axis xyz="0 1 0" rpy="0 0 0" />
-<joint_properties damping="0.0" friction="0.0" />
-</joint>
-<link name="laser_link">
-  <visual>
-    <geometry>
-      <box size="0.05 0.05 0.05"/>
-    </geometry>
-    <material name="black">
-      <color rgba="0.0 0.0 0.0 1.0"/>
-    </material>
-  </visual>
-  <collision>
-    <geometry>
-      <box size="0.05 0.05 0.05"/>
-    </geometry>
-  </collision>
-  <inertial>
-    <mass value="0.1"/>
-    <origin xyz="0 0 0.025" rpy="0 0 0"/>
-    <inertia ixx="0.0001" ixy="0" ixz="0" iyy="0.0001" iyz="0" izz="0.0001"/>
-  </inertial>
-</link>
-<joint name="laser_joint" type="fixed">
-  <parent link="chassis"/>
-  <child link="laser_link"/>
-  <origin xyz="0.0 0 0.05" rpy="0 0 0"/>
-</joint>
-<!-- <gazebo>
-    <plugin filename="gz-sim-sensors-system" name="gz::sim::systems::Sensors">
-    <render_engine>ogre2</render_engine>
-    </plugin>
-</gazebo> -->
-<gazebo reference="laser_link">
-  <sensor name="my_lidar" type="gpu_lidar">
-      <frame_id>laser_link</frame_id>
-      <topic>/lidar</topic>
-      <update_rate>10</update_rate>
-      <visualize>true</visualize>
-      <lidar>
-        <scan>
-          <horizontal>
-            <samples>360</samples>
-            <resolution>1</resolution>
-            <min_angle>-3.14159</min_angle>
-            <max_angle>3.14159</max_angle>
-          </horizontal>
-        </scan>
-        <range>
-          <min>0.1</min>    <max>10.0</max>   <resolution>0.01</resolution>
-        </range>
-        <noise>
-          <type>gaussian</type>
-          <mean>0.0</mean>
-          <stddev>0.01</stddev>
-        </noise>
-      </lidar>
-  </sensor>
-</gazebo>
-<gazebo>
-    <plugin filename="gz_ros2_control-system" name="gz_ros2_control::GazeboSimROS2ControlPlugin">
-        <parameters>$(find autonomous_task_4)/config/diff_drive.yaml</parameters>
-    </plugin>
-</gazebo>
-<!-- STEP 1: ADD THIS <ros2_control> TAG -->
-  <ros2_control name="GazeboSystem" type="system">
-    <hardware>
-      <!-- This is the new plugin for Gazebo Sim -->
-      <plugin>gz_ros2_control/GazeboSimSystem</plugin>
-    </hardware>
-    <!-- Define your left wheel joint for ros2_control -->
-    <joint name="left_wheel_hinge">
-      <command_interface name="velocity">
-        <param name="min">-10</param>
-        <param name="max">10</param>
-      </command_interface>
-      <state_interface name="velocity"/>
-      <state_interface name="position"/>
+    <!-- Robot Parameters -->
+    <xacro:property name="PI" value="3.14159265"/>
+    <xacro:property name="body_length" value="0.5"/>
+    <xacro:property name="body_width" value="0.3"/>
+    <xacro:property name="body_height" value="0.1"/>
+    <xacro:property name="body_density" value="7850.0"/> <!-- Steel -->
+    <xacro:property name="body_mass" value="${body_density * body_length * body_height * body_width}"/>
+    <xacro:property name="body_inertia_x" value="${1.0/12.0 * body_mass * (body_height*body_height + body_width*body_width)}"/>
+    <xacro:property name="body_inertia_y" value="${1.0/12.0 * body_mass * (body_length*body_length + body_height*body_height)}"/>
+    <xacro:property name="body_inertia_z" value="${1.0/12.0 * body_mass * (body_length*body_length + body_width*body_width)}"/>
+    <xacro:property name="wheel_radius" value="0.1"/>
+    <xacro:property name="wheel_width" value="0.05"/>
+    <xacro:property name="wheel_separation" value="${body_width + wheel_width}"/>
+    <xacro:property name="wheel_offset" value="${body_length/2 - wheel_radius}"/>
+    <xacro:property name="wheel_density" value="900"/> <!-- Ruber -->
+    <xacro:property name="wheel_mass" value="${wheel_density * PI * wheel_radius * wheel_radius * wheel_width}"/>
+    <xacro:property name="wheel_inertia_x" value="${1.0/12.0 * wheel_mass * (3*wheel_radius*wheel_radius + wheel_width*wheel_width)}"/>
+    <xacro:property name="wheel_inertia_y" value="${1.0/12.0 * wheel_mass * (3*wheel_radius*wheel_radius + wheel_width*wheel_width)}"/>
+    <xacro:property name="wheel_inertia_z" value="${1.0/2.0 * wheel_mass * wheel_radius * wheel_radius}"/>
+    <xacro:property name="caster_radius" value="0.1"/>
+    <xacro:property name="caster_offset" value="${body_length/2 - caster_radius}"/>
+    <xacro:property name="caster_density" value="0.1"/>
+    <xacro:property name="caster_mass" value="${caster_density * 4.0/3.0 * PI * caster_radius * caster_radius * caster_radius}"/>
+    <xacro:property name="caster_inertia_x" value="${2.0/5.0 * caster_mass * caster_radius * caster_radius}"/>
+    <xacro:property name="caster_inertia_y" value="${2.0/5.0 * caster_mass * caster_radius * caster_radius}"/>
+    <xacro:property name="caster_inertia_z" value="${2.0/5.0 * caster_mass * caster_radius * caster_radius}"/>
+    <!-- Control Parameters -->
+    <xacro:property name="max_linear_acceleration" value="10"/>
+    <!-- Links -->
+    <!-- Body Link -->
+    <link name="body_link">
+        <visual>
+            <origin xyz="0.0 0.0 0.0" rpy="0.0 0.0 0.0"/>
+            <geometry>
+                <box size="${body_length} ${body_width} ${body_height}"/>
+            </geometry>
+            <material name="body_material">
+                <color rgba="0.25 0.25 0.25 1.0"/>
+            </material>
+        </visual>
+        <collision>
+            <origin xyz="0.0 0.0 0.0" rpy="0.0 0.0 0.0"/>
+            <geometry>
+                <box size="${body_length} ${body_width} ${body_height}"/>
+            </geometry>
+        </collision>
+        <inertial>
+            <mass value="10"/>
+            <inertia ixx="${body_inertia_x}" ixy="0.0" ixz="0.0" iyy="${body_inertia_y}" iyz="0" izz="${body_inertia_z}"/>
+            <origin xyz="0 0 0" rpy="0 0 0"/>
+        </inertial>
+    </link>
+    <!-- Left Wheel -->
+    <link name="left_wheel_link">
+        <visual>
+            <origin xyz="0.0 0.0 0.0" rpy="1.570795 0.0 0.0"/>
+            <geometry>
+                <cylinder radius="${wheel_radius}" length="${wheel_width}"/>
+            </geometry>
+            <material name="wheel_material">
+                <color rgba="0.0 0.0 0.0 1.0"/>
+            </material>
+        </visual>
+        <collision>
+            <origin xyz="0.0 0.0 0.0" rpy="1.570795 0.0 0.0"/>
+            <geometry>
+                <cylinder radius="${wheel_radius}" length="${wheel_width}"/>
+            </geometry>
+        </collision>
+        <inertial>
+            <mass value="2"/>
+            <inertia ixx="${wheel_inertia_x}" ixy="0.0" ixz="0.0" iyy="${wheel_inertia_y}" iyz="0" izz="${wheel_inertia_z}"/>
+            <origin xyz="0.0 0.0 0.0" rpy="1.570795 0.0 0.0"/>
+        </inertial>
+    </link>
+    <!-- Right Wheel -->
+    <link name="right_wheel_link">
+        <visual>
+            <origin xyz="0.0 0.0 0.0" rpy="1.570795 0.0 0.0"/>
+            <geometry>
+                <cylinder radius="${wheel_radius}" length="${wheel_width}"/>
+            </geometry>
+            <material name="wheel_material">
+                <color rgba="0.0 0.0 0.0 1.0"/>
+            </material>
+        </visual>
+        <collision>
+            <origin xyz="0.0 0.0 0.0" rpy="1.570795 0.0 0.0"/>
+            <geometry>
+                <cylinder radius="${wheel_radius}" length="${wheel_width}"/>
+            </geometry>
+        </collision>
+        <inertial>
+            <mass value="2"/>
+            <inertia ixx="${wheel_inertia_x}" ixy="0.0" ixz="0.0" iyy="${wheel_inertia_y}" iyz="0" izz="${wheel_inertia_z}"/>
+            <origin xyz="0.0 0.0 0.0" rpy="1.570795 0.0 0.0"/>
+        </inertial>
+    </link>
+    <!-- Caster Wheel -->
+    <link name="caster_link">
+        <visual>
+            <origin xyz="0.0 0.0 0.0" rpy="0.0 0.0 0.0"/>
+            <geometry>
+                <sphere radius="${caster_radius}"/>
+            </geometry>
+            <material name="caster_material">
+                <color rgba="0.0 0.0 0.0 1.0"/>
+            </material>
+        </visual>
+        <collision>
+            <origin xyz="0.0 0.0 0.0" rpy="0.0 0.0 0.0"/>
+            <geometry>
+                <sphere radius="${caster_radius}"/>
+            </geometry>
+        </collision>
+        <inertial>
+            <mass value="0.5"/>
+            <inertia ixx="${caster_inertia_x}" ixy="0.0" ixz="0.0" iyy="${caster_inertia_y}" iyz="0" izz="${caster_inertia_z}"/>
+            <origin xyz="0 0 0" rpy="0 0 0"/>
+        </inertial>
+    </link>
+    <!-- Joints -->
+    <!-- Left Wheel Joint -->
+    <joint name="left_wheel_joint" type="continuous">
+        <origin xyz="-${wheel_offset} ${wheel_separation/2} -${wheel_radius/2}" rpy="0 0 0"/>
+        <parent link="body_link"/>
+        <child link="left_wheel_link"/>
+        <axis xyz="0 1 0"/>
+        <limit effort="100" velocity="10.0"/>
+        <dynamics damping="0.1" friction="0.1"/>
     </joint>
-    <!-- Define your right wheel joint for ros2_control -->
-    <joint name="right_wheel_hinge">
-      <command_interface name="velocity">
-        <param name="min">-10</param>
-        <param name="max">10</param>
-      </command_interface>
-      <state_interface name="velocity"/>
-      <state_interface name="position"/>
+    <!-- Right Wheel Joint -->
+    <joint name="right_wheel_joint" type="continuous">
+        <origin xyz="-${wheel_offset} ${-wheel_separation/2} -${wheel_radius/2}" rpy="0 0 0"/>
+        <parent link="body_link"/>
+        <child link="right_wheel_link"/>
+        <axis xyz="0 1 0"/>
+        <limit effort="100" velocity="10.0"/>
+        <dynamics damping="0.1" friction="0.1"/>
     </joint>
-  </ros2_control>
-  <!-- <gazebo reference="chassis">
-    <disableFixedJointLumping>true</disableFixedJointLumping>
-  </gazebo> -->
-  <!-- ========================================== -->
+    <!-- Caster Wheel Joint (fixed) -->
+    <joint name="caster_joint" type="fixed">
+        <origin xyz="${caster_offset} 0 -${caster_radius/2}" rpy="0 0 0"/>
+        <parent link="body_link"/>
+        <child link="caster_link"/>
+    </joint>
+    <!-- Gazebo Parameters -->
+    <gazebo reference="body_link">
+        <mu1>1.0</mu1>
+        <mu2>1.0</mu2>
+    </gazebo>
+    <gazebo reference="right_wheel_link">
+        <mu1>1.0</mu1>
+        <mu2>1.0</mu2>
+    </gazebo>
+    <gazebo reference="left_wheel_link">
+        <mu1>1.0</mu1>
+        <mu2>1.0</mu2>
+    </gazebo>
+    <gazebo reference="caster_link">
+        <mu1>0.000001</mu1>
+        <mu2>0.000001</mu2>
+    </gazebo>
+    <!-- Gazebo Plugins -->
+    <gazebo>
+        <plugin filename="gz-sim-diff-drive-system" name="gz::sim::systems::DiffDrive">
+            <right_joint>right_wheel_joint</right_joint>
+            <left_joint>left_wheel_joint</left_joint>
+            <wheel_separation>${wheel_separation}</wheel_separation>
+            <wheel_radius>${wheel_radius}</wheel_radius>
+            <max_linear_acceleration>${max_linear_acceleration}</max_linear_acceleration>
+            <odom_publish_frequency>100</odom_publish_frequency>
+            <topic>cmd_vel</topic>
+            <odom_topic>odom</odom_topic>
+        </plugin>
+        <plugin filename="gz-sim-joint-state-publisher-system" name="gz::sim::systems::JointStatePublisher">
+            <topic>joint_states</topic>
+            <joint_name>right_wheel_joint</joint_name>
+            <joint_name>left_wheel_joint</joint_name>
+        </plugin>
+    </gazebo>
+    <!-- ========================================== -->
   <!--                SENSORS                     -->
   <!-- ========================================== -->
@@ -222,7 +200,7 @@
   </link>
   <joint name="front_camera_joint" type="fixed">
-    <parent link="chassis" />
+    <parent link="body_link" />
     <child link="front_camera_link" />
-    <origin xyz="0.15 0 0.1" rpy="0 0 0" />
+    <origin xyz="0.20 0 0.1" rpy="0 0 0" />
   </joint>
   <!-- Gazebo Harmonic Sensor Definition -->
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